Commit message: Add files via upload

File: uuv_simulator/rov/urdf/ROV.urdf (robot description, URDF)
Before this commit: robot ROV, 3 links, 2 joints
Links:
- removed link link1
- added link base_link, mass 0.00001; collision sphere radius=0.3; visual sphere radius=0.3
- added link thruster0, mass 0.00001; collision cylinder length=0.1 radius=0.1; visual cylinder length=0.1 radius=0.1
- added link thruster1, mass 0.00001; collision cylinder length=0.1 radius=0.1; visual cylinder length=0.1 radius=0.1
- added link thruster2, mass 0.00001; collision cylinder length=0.1 radius=0.1; visual cylinder length=0.1 radius=0.1
- added link thruster3, mass 0.00001; collision cylinder length=0.1 radius=0.1; visual cylinder length=0.1 radius=0.1
- added link thruster4, mass 0.00001; collision cylinder length=0.1 radius=0.1; visual cylinder length=0.1 radius=0.1
- added link thruster5, mass 0.00001; collision cylinder length=0.1 radius=0.1; visual cylinder length=0.1 radius=0.1
- link link2: geometry collision box size=0.5 0.3 0.5; visual box size=0.5 0.3 0.5
Joints:
- added joint thruster_joint0: type continuous, parent base_link, child thruster0, origin xyz=0.15 0.22 0.15 rpy=0 0 -0.79, axis 0.9 0.15 0
- added joint thruster_joint1: type continuous, parent base_link, child thruster1, origin xyz=-0.15 0.22 0.15 rpy=0 0 0.79, axis 0.9 0.15 0
- added joint thruster_joint2: type continuous, parent base_link, child thruster2, origin xyz=0.15 -0.22 0.15 rpy=0 0 0.79, axis 0.9 0.15 0
- added joint thruster_joint3: type continuous, parent base_link, child thruster3, origin xyz=-0.15 -0.22 0.15 rpy=0 0 -0.79, axis 0.9 0.15 0
- added joint thruster_joint4: type continuous, parent base_link, child thruster4, origin xyz=0.35 0.25 0.23 rpy=0 1.57 0, axis 0.9 0.15 0
- added joint thruster_joint5: type continuous, parent base_link, child thruster5, origin xyz=0.65 -0.25 0.23 rpy=0 1.57 0, axis 0.9 0.15 0
- joint joint1: parent link1 -> base_link
- joint joint2: parent link1 -> base_link

Commit message: Add files via upload

File: uuv_simulator/rov/urdf/ROV.urdf (robot description, URDF)
Before this commit: robot ROV, 9 links, 8 joints
Links:
- added link thruster6, mass 0.00001; collision cylinder length=0.1 radius=0.1; visual cylinder length=0.1 radius=0.1
- added link thruster7, mass 0.00001; collision cylinder length=0.1 radius=0.1; visual cylinder length=0.1 radius=0.1
Joints:
- added joint thruster_joint6: type continuous, parent base_link, child thruster6, origin xyz=0.35 -0.25 0.23 rpy=0 1.57 0, axis 0.9 0.15 0
- added joint thruster_joint7: type continuous, parent base_link, child thruster7, origin xyz=0.65 0.25 0.23 rpy=0 1.57 0, axis 0.9 0.15 0
